File: Main-Board/AUV_Controller/AUV_Controller.kicad_sch (KiCad schematic)
At the start: 0 parts

Commit message: menambah board teensy pada projek
Parts:
- added A1: TEENSY_4.1, TEENSY 4.1:TEENSY_LONG_EXT, symbol TEENSY_4.1:TEENSY_4.1
Connections:
- new net: A1.3V3 (3.3V), A1.3V3@2 (3.3V), A1.3V3@3 (3.3V)
- new net: A1.AGND/GND (GND), A1.GND, A1.GND@2 (GND)

Commit message: test
Parts:
- added J1, J2, J3, J4: Conn_01x04_Pin, Connector_JST:JST_EH_S4B-EH_1x04_P2.50mm_Horizontal, symbol Connector:Conn_01x04_Pin
- A1: footprint TEENSY 4.1:TEENSY_LONG_EXT -> TEENSY_4.1:TEENSY_LONG_EXT
